Commit message: Created_core URDF

File: description/robot_core.xacro (robot description, xacro)
@@ -17,11 +17,11 @@
     <link name="base_link">
     </link>
-    <!-- frame LINK -->
-    <joint name="frame_joint" type="fixed">
+    <!-- chassis LINK -->
+    <joint name="chassis_joint" type="fixed">
         <parent link="base_link"/>
-        <child link="frame"/>
+        <child link="chassis"/>
         <origin xyz="-0.1 0 0"/>
     </joint>
-    <link name="frame">
+    <link name="chassis">
         <visual>
             <origin xyz="0.15 0 0.075"/>
@@ -41,5 +41,5 @@
         </xacro:inertial_box>
     </link>
-    <gazebo reference="frame">
+    <gazebo reference="chassis">
         <material>Gazebo/White</material>
     </gazebo>
@@ -98,5 +98,5 @@
     <!-- CASTER WHEEL LINK -->
     <joint name="caster_wheel_joint" type="fixed">
-        <parent link="frame"/>
+        <parent link="chassis"/>
         <child link="caster_wheel"/>
         <origin xyz="0.24 0 0"/>
